Commit message: fix issue with loading mesh files in rviz

File: intel_aero_description/urdf/multirotor_base.xacro (robot description, xacro)
@@ -35,5 +35,5 @@
         <origin xyz="0 0 0" rpy="0 0 0" />
         <geometry>
-          <mesh filename="$(find intel_aero_description)/meshes/${mesh_file}"
+          <mesh filename="file://$(find intel_aero_description)/meshes/${mesh_file}"
             scale="${mesh_scale}" />
           <!-- <box size="${body_width} ${body_width} ${body_height}"/> --> <!-- [m] [m] [m] -->
@@ -95,5 +95,5 @@
           <!-- <cylinder length="0.005" radius="${radius_rotor}"/> --> <!-- [m] -->
           <!-- <mesh filename="package://rotors_description/meshes/propeller_${direction}.dae" -->
-          <mesh filename="$(find intel_aero_description)/meshes/${mesh}_${direction}.dae"
+            <mesh filename="file://$(find intel_aero_description)/meshes/${mesh}_${direction}.dae"
             scale="${mesh_scale}" />
           <!-- <box size="${2*radius_rotor} 0.01 0.005"/> -->
