Commit message: Swith to libgazebo_ros_openni_kinect.so plugin
Remove dependency on realsense_gazebo_plugin package that does not
properly handle ROS node namespacing
Create xacro file for intel r200 camera using
libgazebo_ros_openni_kinect.so plugin to provide depth and color images

File: intel_aero_description/urdf/intel_aero.xacro (robot description, xacro)
@@ -1,13 +1,13 @@
 <?xml version="1.0" ?>
 <robot name="intel_aero" xmlns:xacro="http://ros.org/wiki/xacro">
-  <!-- include iris_base provided with PX4 package -->
+  <!-- iris_base -->
   <xacro:include filename="$(find intel_aero_description)/urdf/iris_base.xacro" />
-  <!-- load rs200 macro from realsense_gazebo_plugin package -->
-  <xacro:include filename="$(find realsense_gazebo_plugin)/urdf/realsense-RS200.macro.xacro" />
-  <!-- create instance of RS200 and attach it to the iris -->
-  <xacro:realsense-rs200 />
+  <!-- realsense r200 macro -->
+  <xacro:include filename="$(find intel_aero_description)/urdf/r200.macro.xacro" />
+  <!-- create instance of r200 and attach it to the iris -->
+  <xacro:realsense_r200 />
   <joint name="realsense_joint" type="fixed">
     <parent link="base_link" />
-    <child link="rs200_camera" />
+    <child link="camera_link" />
     <origin ryp="0 0 0" xyz="0.101 0 0" />
   </joint>

Commit message: add world frame to tf tree and use tf2 to convert when planning

File: intel_aero_description/urdf/intel_aero.xacro (robot description, xacro)
@@ -2,4 +2,5 @@
 <robot name="intel_aero" xmlns:xacro="http://ros.org/wiki/xacro">
   <xacro:arg name='namespace' default='' />
+  <xacro:arg name='max_range' default='10.0'/>
   <!-- iris_base -->
   <xacro:include filename="$(find intel_aero_description)/urdf/iris_base.xacro" />
@@ -7,4 +8,6 @@
   <xacro:include filename="$(find intel_aero_description)/urdf/r200.macro.xacro" />
   <!-- create instance of r200 and attach it to the iris -->
-  <xacro:realsense_r200 namespace="$(arg namespace)" parent_link="$(arg namespace)/base_link" />
+  <xacro:realsense_r200 namespace="$(arg namespace)"
+                        parent_link="$(arg namespace)/base_link"
+                        max_range="$(arg max_range)"/>
 </robot>

File: intel_aero_description/urdf/r200.macro.xacro (robot description, xacro)
@@ -7,5 +7,5 @@
   <xacro:property name="r200_cam_depth_offset" value="0.01"/>
   <!-- camera macro -->
-  <xacro:macro name="realsense_r200" params="namespace parent_link">
+  <xacro:macro name="realsense_r200" params="namespace parent_link max_range">
     <!-- Camera joint -->
     <joint name="${namespace}/camera_joint" type="fixed">
@@ -74,6 +74,6 @@
           </depth_camera>
           <clip>
-            <near>0.5</near>
-            <far>10.0</far>
+            <near>0.25</near>
+            <far>${max_range}</far>
           </clip>
         </camera>
