Commit message: update urdf files to allow for tf frame prefix

File: intel_aero_description/urdf/component_snippets.xacro (robot description, xacro)
@@ -24,6 +24,6 @@
         <robotNamespace>${namespace}</robotNamespace>
         <bagFileName>${bag_file}</bagFileName>
-        <linkName>base_link</linkName>
-        <frameId>base_link</frameId>
+        <linkName>${namespace}/base_link</linkName>
+        <frameId>${namespace}/base_link</frameId>
         <commandAttitudeThrustSubTopic>command/attitude</commandAttitudeThrustSubTopic>
         <commandAttitudeThrustPubTopic>command/attitude</commandAttitudeThrustPubTopic>
@@ -37,5 +37,5 @@
       horizontal_fov image_width image_height image_format min_distance
       max_distance noise_mean noise_stddev enable_visual *cylinder *origin">
-    <link name="${namespace}/camera_${camera_suffix}_link">
+    <link name="$(arg namespace)/camera_${camera_suffix}_link">
       <collision>
         <origin xyz="0 0 0" rpy="0 0 0" />
@@ -128,5 +128,8 @@
   </xacro:macro>
   <!-- Macro to add the mavlink interface. -->
-  <xacro:macro name="mavlink_interface_macro" params="namespace imu_sub_topic gps_sub_topic mavlink_addr mavlink_udp_port serial_enabled serial_device baudrate qgc_addr qgc_udp_port hil_mode hil_state_level vehicle_is_tailsitter">
+  <xacro:macro name="mavlink_interface_macro"
+    params="namespace imu_sub_topic gps_sub_topic mavlink_addr mavlink_udp_port
+        serial_enabled serial_device baudrate qgc_addr qgc_udp_port hil_mode
+        hil_state_level vehicle_is_tailsitter">
     <gazebo>
       <plugin name="mavlink_interface" filename="libgazebo_mavlink_interface.so">
@@ -265,5 +268,5 @@
     <joint name="${namespace}/imu${imu_suffix}_joint" type="revolute">
       <xacro:insert_block name="origin" />
-      <parent link="${parent_link}" />
+      <parent link="${namespace}/${parent_link}" />
       <child link="${namespace}/imu${imu_suffix}_link" />
       <limit upper="0" lower="0" effort="0" velocity="0" />
@@ -274,5 +277,5 @@
            https://github.com/ethz-asl/kalibr/wiki/IMU-Noise-Model-and-Intrinsics -->
         <robotNamespace>${namespace}</robotNamespace> <!-- (string, required): ros namespace in which the messages are published -->
-        <linkName>${namespace}/imu${imu_suffix}_link</linkName> <!-- (string, required): name of the body which holds the IMU sensor -->
+          <linkName>${namespace}/imu${imu_suffix}_link</linkName> <!-- (string, required): name of the body which holds the IMU sensor -->
         <imuTopic>${imu_topic}</imuTopic> <!-- (string): name of the sensor output topic and prefix of service names (defaults to imu) -->
         <gyroscopeNoiseDensity>${gyroscope_noise_density}</gyroscopeNoiseDensity> <!-- Gyroscope noise density (two-sided spectrum) [rad/s/sqrt(Hz)] -->
@@ -287,5 +290,5 @@
     </gazebo>
   </xacro:macro>
-<!-- Macro to add a generic odometry sensor. -->
+  <!-- Macro to add a generic odometry sensor. -->
   <xacro:macro name="odometry_plugin_macro"
     params="

File: intel_aero_description/urdf/intel_aero.xacro (robot description, xacro)
@@ -1,4 +1,5 @@
 <?xml version="1.0" ?>
 <robot name="intel_aero" xmlns:xacro="http://ros.org/wiki/xacro">
+  <xacro:arg name='namespace' default='' />
   <!-- iris_base -->
   <xacro:include filename="$(find intel_aero_description)/urdf/iris_base.xacro" />
@@ -6,9 +7,4 @@
   <xacro:include filename="$(find intel_aero_description)/urdf/r200.macro.xacro" />
   <!-- create instance of r200 and attach it to the iris -->
-  <xacro:realsense_r200 />
-  <joint name="realsense_joint" type="fixed">
-    <parent link="base_link" />
-    <child link="camera_link" />
-    <origin ryp="0 0 0" xyz="0.101 0 0" />
-  </joint>
+  <xacro:realsense_r200 namespace="$(arg namespace)" parent_link="base_link" />
 </robot>

File: intel_aero_description/urdf/iris.xacro (robot description, xacro)
@@ -2,5 +2,4 @@
 <robot name="iris" xmlns:xacro="http://ros.org/wiki/xacro">
   <!-- Properties -->
-  <xacro:property name="namespace" value="" />
   <xacro:property name="rotor_velocity_slowdown_sim" value="10" />
   <xacro:property name="mesh_file" value="iris.stl" />
@@ -44,5 +43,5 @@
   <!-- Instantiate multirotor_base_macro once -->
   <xacro:multirotor_base_macro
-    robot_namespace="${namespace}"
+    robot_namespace="$(arg namespace)"
     mass="${mass}"
     body_width="${body_width}"
@@ -56,5 +55,5 @@
   <!-- Instantiate rotors -->
   <xacro:vertical_rotor
-    robot_namespace="${namespace}"
+    robot_namespace="$(arg namespace)"
     suffix="front_right"
     direction="ccw"
@@ -77,5 +76,5 @@
   </xacro:vertical_rotor>
   <xacro:vertical_rotor
-    robot_namespace="${namespace}"
+    robot_namespace="$(arg namespace)"
     suffix="back_left"
     direction="ccw"
@@ -97,5 +96,5 @@
     <xacro:insert_block name="rotor_inertia" />
   </xacro:vertical_rotor>
-  <xacro:vertical_rotor robot_namespace="${namespace}"
+  <xacro:vertical_rotor robot_namespace="$(arg namespace)"
     suffix="front_left"
     direction="cw"
@@ -117,5 +116,5 @@
     <xacro:insert_block name="rotor_inertia" />
   </xacro:vertical_rotor>
-  <xacro:vertical_rotor robot_namespace="${namespace}"
+  <xacro:vertical_rotor robot_namespace="$(arg namespace)"
     suffix="back_right"
     direction="cw"

File: intel_aero_description/urdf/iris_base.xacro (robot description, xacro)
@@ -28,5 +28,5 @@
   <xacro:if value="$(arg enable_wind)">
     <xacro:wind_plugin_macro
-        namespace="${namespace}"
+        namespace="$(arg namespace)"
         wind_direction="0 0 1"
         wind_force_mean="0.7"
@@ -38,32 +38,28 @@
         />
   </xacro:if>
-    <!-- Instantiate gps plugin. -->
-  <xacro:gps_plugin_macro
-    namespace="${namespace}"
-    gps_noise="true"
-    >
-  </xacro:gps_plugin_macro>
+  <!-- Instantiate gps plugin. -->
+  <xacro:gps_plugin_macro namespace="$(arg namespace)" gps_noise="true" />
+  <!-- Instantiate mavlink telemetry interface. -->
   <xacro:if value="$(arg enable_mavlink_interface)">
-  <!-- Instantiate mavlink telemetry interface. -->
-  <xacro:mavlink_interface_macro
-    namespace="${namespace}"
-    imu_sub_topic="/imu"
-    gps_sub_topic="/gps"
-    mavlink_addr="$(arg mavlink_addr)"
-    mavlink_udp_port="$(arg mavlink_udp_port)"
-    serial_enabled="$(arg serial_enabled)"
-    serial_device="$(arg serial_device)"
-    baudrate="$(arg baudrate)"
-    qgc_addr="$(arg qgc_addr)"
-    qgc_udp_port="$(arg qgc_udp_port)"
-    hil_mode="$(arg hil_mode)"
-    hil_state_level="$(arg hil_state_level)"
-    vehicle_is_tailsitter="$(arg vehicle_is_tailsitter)"
-    >
-  </xacro:mavlink_interface_macro>
+    <xacro:mavlink_interface_macro
+      namespace="$(arg namespace)"
+      imu_sub_topic="/imu"
+      gps_sub_topic="/gps"
+      mavlink_addr="$(arg mavlink_addr)"
+      mavlink_udp_port="$(arg mavlink_udp_port)"
+      serial_enabled="$(arg serial_enabled)"
+      serial_device="$(arg serial_device)"
+      baudrate="$(arg baudrate)"
+      qgc_addr="$(arg qgc_addr)"
+      qgc_udp_port="$(arg qgc_udp_port)"
+      hil_mode="$(arg hil_mode)"
+      hil_state_level="$(arg hil_state_level)"
+      vehicle_is_tailsitter="$(arg vehicle_is_tailsitter)"
+      >
+    </xacro:mavlink_interface_macro>
   </xacro:if>
   <!-- Mount an ADIS16448 IMU. -->
   <xacro:imu_plugin_macro
-    namespace="${namespace}"
+    namespace="$(arg namespace)"
     imu_suffix=""
     parent_link="base_link"
@@ -85,5 +81,5 @@
     <!-- Mount an IMU providing ground truth. -->
     <xacro:imu_plugin_macro
-      namespace="${namespace}"
+      namespace="$(arg namespace)"
       imu_suffix="gt"
       parent_link="base_link"
@@ -104,5 +100,5 @@
     <!-- Mount a generic odometry sensor providing ground truth. -->
     <xacro:odometry_plugin_macro
-      namespace="${namespace}/ground_truth"
+      namespace="$(arg namespace)/ground_truth"
       odometry_sensor_suffix="gt"
       parent_link="base_link"
@@ -136,5 +132,5 @@
     <!-- Instantiate a logger -->
     <xacro:bag_plugin_macro
-      namespace="${namespace}"
+      namespace="$(arg namespace)"
       bag_file="$(arg log_file)"
       rotor_velocity_slowdown_sim="${rotor_velocity_slowdown_sim}"

File: intel_aero_description/urdf/multirotor_base.xacro (robot description, xacro)
@@ -20,11 +20,11 @@
   <xacro:macro name="multirotor_base_macro"
     params="robot_namespace mass body_width body_height mesh_file mesh_scale color *inertia">
-    <link name="base_link"></link>
-    <joint name="base_joint" type="fixed">
+    <link name="${robot_namespace}/base_link"></link>
+    <joint name="${robot_namespace}/base_joint" type="fixed">
       <origin xyz="0 0 0" rpy="0 0 0" />
-      <parent link="base_link" />
-      <child link="base_link_inertia" />
+      <parent link="${robot_namespace}/base_link" />
+      <child link="${robot_namespace}/base_link_inertia" />
     </joint>
-    <link name="base_link_inertia">
+    <link name="${robot_namespace}/base_link_inertia">
       <inertial>
         <mass value="${mass}" />  <!-- [kg] -->
@@ -51,9 +51,9 @@
       <plugin filename="libgazebo_multirotor_base_plugin.so" name="rosbag">
         <robotNamespace>${robot_namespace}</robotNamespace>
-        <linkName>base_link</linkName>
+        <linkName>${robot_namespace}/base_link</linkName>
         <rotorVelocitySlowdownSim>${rotor_velocity_slowdown_sim}</rotorVelocitySlowdownSim>
       </plugin>
     </gazebo>
-    <gazebo reference="base_link">
+    <gazebo reference="${robot_namespace}/base_link">
       <material>Gazebo/${color}</material>
       <collision name='base_link_inertia_collision'>
@@ -75,16 +75,16 @@
   <xacro:macro name="vertical_rotor"
     params="robot_namespace suffix direction motor_constant moment_constant parent mass_rotor radius_rotor time_constant_up time_constant_down max_rot_velocity motor_number rotor_drag_coefficient rolling_moment_coefficient color mesh mesh_scale *origin *inertia">
-    <joint name="rotor_${motor_number}_joint" type="continuous">
+    <joint name="${robot_namespace}/rotor_${motor_number}_joint" type="continuous">
       <xacro:insert_block name="origin" />
       <axis xyz="0 0 1" />
       <!-- TODO(ff): not currently set because it's not yet supported -->
       <!-- <limit effort="2000" velocity="${max_rot_velocity}" /> -->
-      <parent link="${parent}" />
-      <child link="rotor_${motor_number}" />
+      <parent link="${robot_namespace}/${parent}" />
+      <child link="${robot_namespace}/rotor_${motor_number}" />
     </joint>
     <!-- TODO(ff): not currently set because it's not yet supported -->
     <!-- <gazebo reference="rotor_${motor_number}_joint"> <axis> <xyz>0 0 1</xyz>
       <limit> <velocity> ${max_rot_velocity} </velocity> </limit> </axis> </gazebo> -->
-    <link name="rotor_${motor_number}">
+    <link name="${robot_namespace}/rotor_${motor_number}">
       <inertial>
         <mass value="${mass_rotor}" /> <!-- [kg] -->
@@ -109,6 +109,6 @@
       <plugin name="${suffix}_motor_model" filename="libgazebo_motor_model.so">
         <robotNamespace>${robot_namespace}</robotNamespace>
-        <jointName>rotor_${motor_number}_joint</jointName>
-        <linkName>rotor_${motor_number}</linkName>
+        <jointName>${robot_namespace}/rotor_${motor_number}_joint</jointName>
+        <linkName>${robot_namespace}/rotor_${motor_number}</linkName>
         <turningDirection>${direction}</turningDirection>
         <timeConstantUp>${time_constant_up}</timeConstantUp>
@@ -136,5 +136,5 @@
       </plugin>
     </gazebo>
-    <gazebo reference="rotor_${motor_number}">
+    <gazebo reference="${robot_namespace}/rotor_${motor_number}">
       <material>Gazebo/${color}</material>
     </gazebo>

File: intel_aero_description/urdf/r200.macro.xacro (robot description, xacro)
@@ -6,7 +6,14 @@
   <xacro:property name="r200_cam_rgb_pz" value="0.013"/>
   <xacro:property name="r200_cam_depth_offset" value="0.01"/>
-  <xacro:macro name="realsense_r200">
+  <!-- camera macro -->
+  <xacro:macro name="realsense_r200" params="namespace parent_link">
+    <!-- Camera joint -->
+    <joint name="${namespace}/camera_joint" type="fixed">
+      <parent link="${namespace}/${parent_link}" />
+      <child link="${namespace}/camera_link" />
+      <origin ryp="0 0 0" xyz="0.101 0 0" />
+    </joint>
     <!-- Camera link -->
-    <link name="camera_link">
+    <link name="${namespace}/camera_link">
       <visual>
         <origin rpy="0 0 0" xyz="0 0 0"/>
@@ -27,31 +34,31 @@
     </link>
     <!-- RGB joints & links -->
-    <link name="camera_rgb_frame"/>
-    <joint name="camera_rgb_joint" type="fixed">
+    <link name="${namespace}/camera_rgb_frame"/>
+    <joint name="${namespace}/camera_rgb_joint" type="fixed">
       <origin xyz="${r200_cam_rgb_px} ${r200_cam_rgb_py} ${r200_cam_rgb_pz}" rpy="0 0 0"/>
-      <parent link="camera_link"/>
-      <child link="camera_rgb_frame" />
+      <parent link="${namespace}/camera_link"/>
+      <child link="${namespace}/camera_rgb_frame" />
     </joint>
-    <link name="camera_rgb_optical_frame"/>
-    <joint name="camera_rgb_optical_joint" type="fixed">
+    <link name="${namespace}/camera_rgb_optical_frame"/>
+    <joint name="${namespace}/camera_rgb_optical_joint" type="fixed">
       <origin xyz="0 0 0" rpy="${-pi/2} 0 ${-pi/2}" />
-      <parent link="camera_rgb_frame" />
-      <child link="camera_rgb_optical_frame" />
+      <parent link="${namespace}/camera_rgb_frame" />
+      <child link="${namespace}/camera_rgb_optical_frame" />
     </joint>
     <!-- Depth joints & links -->
-    <link name="camera_depth_frame"/>
-    <joint name="camera_depth_joint" type="fixed">
-        <origin xyz="0 ${r200_cam_depth_offset} 0" rpy="0 0 0" />
-        <parent link="camera_rgb_frame" />
-        <child link="camera_depth_frame" />
+    <link name="${namespace}/camera_depth_frame"/>
+    <joint name="${namespace}/camera_depth_joint" type="fixed">
+      <origin xyz="0 ${r200_cam_depth_offset} 0" rpy="0 0 0" />
+      <parent link="${namespace}/camera_rgb_frame" />
+      <child link="${namespace}/camera_depth_frame" />
     </joint>
-    <link name="camera_depth_optical_frame"/>
-    <joint name="camera_depth_optical_joint" type="fixed">
-        <origin xyz="0 0 0" rpy="${-pi/2} 0 ${-pi/2}" />
-        <parent link="camera_depth_frame" />
-        <child link="camera_depth_optical_frame" />
+    <link name="${namespace}/camera_depth_optical_frame"/>
+    <joint name="${namespace}/camera_depth_optical_joint" type="fixed">
+      <origin xyz="0 0 0" rpy="${-pi/2} 0 ${-pi/2}" />
+      <parent link="${namespace}/camera_depth_frame" />
+      <child link="${namespace}/camera_depth_optical_frame" />
     </joint>
     <!-- Depth camera plugin -->
-    <gazebo reference="camera_link">
+    <gazebo reference="${namespace}/camera_link">
       <sensor type="depth" name="camera">
         <always_on>true</always_on>
@@ -73,4 +80,7 @@
         <plugin name="kinect_camera_controller" filename="libgazebo_ros_openni_kinect.so">
           <cameraName>camera</cameraName>
+          <robotNamespace>${namespace}</robotNamespace>
+          <jointName>${namespace}/camera_joint</jointName>
+          <linkName>${namespace}/camera_link</linkName>
           <alwaysOn>true</alwaysOn>
           <updateRate>0.0</updateRate>
@@ -80,5 +90,5 @@
           <cameraInfoTopicName>rgb/camera_info</cameraInfoTopicName>
           <depthImageCameraInfoTopicName>depth/camera_info</depthImageCameraInfoTopicName>
-          <frameName>camera_depth_optical_frame</frameName>
+          <frameName>${namespace}/camera_depth_optical_frame</frameName>
           <baseline>0.1</baseline>
           <distortion_k1>0.0</distortion_k1>

Commit message: parent parameter should be fully name resolved

File: intel_aero_description/urdf/component_snippets.xacro (robot description, xacro)
@@ -268,5 +268,5 @@
     <joint name="${namespace}/imu${imu_suffix}_joint" type="revolute">
       <xacro:insert_block name="origin" />
-      <parent link="${namespace}/${parent_link}" />
+      <parent link="${parent_link}" />
       <child link="${namespace}/imu${imu_suffix}_link" />
       <limit upper="0" lower="0" effort="0" velocity="0" />
@@ -302,5 +302,5 @@
       image_scale *inertia *origin">
     <!-- odometry link -->
-    <link name="${namespace}/odometry_sensor${odometry_sensor_suffix}_link">
+    <link name="${namespace}/odometry_sensor_${odometry_sensor_suffix}_link">
       <inertial>
         <xacro:insert_block name="inertia" />
@@ -309,8 +309,8 @@
     </link>
     <!-- odometry joint -->
-    <joint name="${namespace}/odometry_sensor${odometry_sensor_suffix}_joint" type="revolute">
+    <joint name="${namespace}/odometry_sensor_${odometry_sensor_suffix}_joint" type="revolute">
       <parent link="${parent_link}" />
       <xacro:insert_block name="origin" />
-      <child link="${namespace}/odometry_sensor${odometry_sensor_suffix}_link" />
+      <child link="${namespace}/odometry_sensor_${odometry_sensor_suffix}_link" />
       <limit upper="0" lower="0" effort="0" velocity="0" />
     </joint>

File: intel_aero_description/urdf/intel_aero.xacro (robot description, xacro)
@@ -7,4 +7,4 @@
   <xacro:include filename="$(find intel_aero_description)/urdf/r200.macro.xacro" />
   <!-- create instance of r200 and attach it to the iris -->
-  <xacro:realsense_r200 namespace="$(arg namespace)" parent_link="base_link" />
+  <xacro:realsense_r200 namespace="$(arg namespace)" parent_link="$(arg namespace)/base_link" />
 </robot>

File: intel_aero_description/urdf/iris.xacro (robot description, xacro)
@@ -60,5 +60,5 @@
     motor_constant="${motor_constant}"
     moment_constant="${moment_constant}"
-    parent="base_link"
+    parent="$(arg namespace)/base_link"
     mass_rotor="${mass_rotor}"
     radius_rotor="${radius_rotor}"
@@ -81,5 +81,5 @@
     motor_constant="${motor_constant}"
     moment_constant="${moment_constant}"
-    parent="base_link"
+    parent="$(arg namespace)/base_link"
     mass_rotor="${mass_rotor}"
     radius_rotor="${radius_rotor}"
@@ -101,5 +101,5 @@
     motor_constant="${motor_constant}"
     moment_constant="${moment_constant}"
-    parent="base_link"
+    parent="$(arg namespace)/base_link"
     mass_rotor="${mass_rotor}"
     radius_rotor="${radius_rotor}"
@@ -121,5 +121,5 @@
     motor_constant="${motor_constant}"
     moment_constant="${moment_constant}"
-    parent="base_link"
+    parent="$(arg namespace)/base_link"
     mass_rotor="${mass_rotor}"
     radius_rotor="${radius_rotor}"

File: intel_aero_description/urdf/iris_base.xacro (robot description, xacro)
@@ -39,5 +39,5 @@
   </xacro:if>
   <!-- Instantiate gps plugin. -->
-  <xacro:gps_plugin_macro namespace="$(arg namespace)" gps_noise="true" />
+  <xacro:gps_plugin_macro namespace="$(arg namespace)" gps_noise="false" />
   <!-- Instantiate mavlink telemetry interface. -->
   <xacro:if value="$(arg enable_mavlink_interface)">
@@ -63,5 +63,5 @@
     namespace="$(arg namespace)"
     imu_suffix=""
-    parent_link="base_link"
+    parent_link="$(arg namespace)/base_link"
     imu_topic="/imu"
     mass_imu_sensor="0.015"
@@ -83,5 +83,5 @@
       namespace="$(arg namespace)"
       imu_suffix="gt"
-      parent_link="base_link"
+      parent_link="$(arg namespace)/base_link"
       imu_topic="ground_truth/imu"
       mass_imu_sensor="0.00001"
@@ -102,5 +102,5 @@
       namespace="$(arg namespace)/ground_truth"
       odometry_sensor_suffix="gt"
-      parent_link="base_link"
+      parent_link="$(arg namespace)/base_link"
       pose_topic="pose"
       pose_with_covariance_topic="pose_with_covariance"

File: intel_aero_description/urdf/multirotor_base.xacro (robot description, xacro)
@@ -23,5 +23,5 @@
     <joint name="${robot_namespace}/base_joint" type="fixed">
       <origin xyz="0 0 0" rpy="0 0 0" />
-      <parent link="${robot_namespace}/base_link" />
+      <parent link="$(arg namespace)/base_link" />
       <child link="${robot_namespace}/base_link_inertia" />
     </joint>
@@ -80,5 +80,5 @@
       <!-- TODO(ff): not currently set because it's not yet supported -->
       <!-- <limit effort="2000" velocity="${max_rot_velocity}" /> -->
-      <parent link="${robot_namespace}/${parent}" />
+      <parent link="${parent}" />
       <child link="${robot_namespace}/rotor_${motor_number}" />
     </joint>

File: intel_aero_description/urdf/r200.macro.xacro (robot description, xacro)
@@ -10,5 +10,5 @@
     <!-- Camera joint -->
     <joint name="${namespace}/camera_joint" type="fixed">
-      <parent link="${namespace}/${parent_link}" />
+      <parent link="${parent_link}" />
       <child link="${namespace}/camera_link" />
       <origin ryp="0 0 0" xyz="0.101 0 0" />
