Commit message: syncing repos

File: intel_aero_description/urdf/component_snippets.xacro (robot description, xacro)
@@ -129,7 +129,10 @@
   <!-- Macro to add the mavlink interface. -->
   <xacro:macro name="mavlink_interface_macro"
-    params="namespace imu_sub_topic gps_sub_topic mavlink_addr mavlink_udp_port
-        serial_enabled serial_device baudrate qgc_addr qgc_udp_port hil_mode
-        hil_state_level vehicle_is_tailsitter">
+               params="namespace imu_sub_topic gps_sub_topic mavlink_addr
+                       mavlink_udp_port mavlink_tcp_port serial_enabled
+                       serial_device baudrate qgc_addr qgc_udp_port hil_mode
+                       hil_state_level vehicle_is_tailsitter
+                       send_vision_estimation send_odometry enable_lockstep
+                       use_tcp">
     <gazebo>
       <plugin name="mavlink_interface" filename="libgazebo_mavlink_interface.so">
@@ -139,4 +142,5 @@
         <mavlink_addr>$(arg mavlink_addr)</mavlink_addr>
         <mavlink_udp_port>$(arg mavlink_udp_port)</mavlink_udp_port>
+        <mavlink_tcp_port>$(arg mavlink_tcp_port)</mavlink_tcp_port>
         <serialEnabled>$(arg serial_enabled)</serialEnabled>
         <serialDevice>$(arg serial_device)</serialDevice>
@@ -147,4 +151,8 @@
         <hil_state_level>$(arg hil_state_level)</hil_state_level>
         <vehicle_is_tailsitter>$(arg vehicle_is_tailsitter)</vehicle_is_tailsitter>
+        <send_vision_estimation>$(arg send_vision_estimation)</send_vision_estimation>
+        <send_odometry>$(arg send_odometry)</send_odometry>
+        <enable_lockstep>$(arg enable_lockstep)</enable_lockstep>
+        <use_tcp>$(arg use_tcp)</use_tcp>
         <motorSpeedCommandPubTopic>/gazebo/command/motor_speed</motorSpeedCommandPubTopic>
         <control_channels>

File: intel_aero_description/urdf/intel_aero.xacro (robot description, xacro)
@@ -1,19 +1,25 @@
 <?xml version="1.0" ?>
 <robot name="intel_aero" xmlns:xacro="http://ros.org/wiki/xacro">
-  <xacro:arg name='namespace' default='' />
-  <xacro:arg name='max_range' default='10.0'/>
+  <xacro:arg name="namespace"        default=""/>
+  <xacro:arg name="max_range"        default="10.0"/>
+  <xacro:arg name="enable_realsense" default="false"/>
+  <xacro:arg name="spawn_only"       default="false"/>
   <!-- iris_base -->
-  <xacro:include filename="$(find intel_aero_description)/urdf/iris_base.xacro" />
-  <!-- realsense r200 macro -->
-  <xacro:include filename="$(find intel_aero_description)/urdf/r200.macro.xacro" />
+  <xacro:include filename="$(find intel_aero_description)/urdf/iris_base.xacro"/>
   <!-- create instance of r200 and attach it to the iris -->
-  <xacro:realsense_r200 namespace="$(arg namespace)"
-                        parent_link="$(arg namespace)/base_link"
-                        max_range="$(arg max_range)"/>
+  <xacro:include filename="$(find intel_aero_description)/urdf/r200.macro.xacro"/>
+  <!-- load realsense plugin for streaming depth/rgb frames -->
+  <xacro:if value="$(arg enable_realsense)">
+    <xacro:realsense_r200 namespace="$(arg namespace)"
+                          parent_link="$(arg namespace)/base_link"
+                          max_range="$(arg max_range)"/>
+  </xacro:if>
   <!-- load plugin for sending velocity commands directly to the quadrotor -->
-  <gazebo>
-    <plugin name="intel_aero_gazebo" filename="libvelocity_control.so">
-      <link_name>$(arg namespace)/base_link</link_name>
-    </plugin>
-  </gazebo>
+  <xacro:if value="$(arg spawn_only)">
+    <gazebo>
+      <plugin name="intel_aero_gazebo" filename="libvelocity_control.so">
+        <link_name>$(arg namespace)/base_link</link_name>
+      </plugin>
+    </gazebo>
+  </xacro:if>
 </robot>

File: intel_aero_description/urdf/iris_base.xacro (robot description, xacro)
@@ -4,137 +4,150 @@
   Is there a reason not to make all properties arguments?
   -->
-  <xacro:arg name='name' default='iris' />
-  <xacro:arg name='mavlink_addr' default='INADDR_ANY' />
-  <xacro:arg name='mavlink_udp_port' default='14560' />
-  <xacro:arg name='serial_enabled' default='false' />
-  <xacro:arg name='serial_device' default='/dev/ttyACM0' />
-  <xacro:arg name='baudrate' default='921600' />
-  <xacro:arg name='qgc_addr' default='INADDR_ANY' />
-  <xacro:arg name='qgc_udp_port' default='14550' />
-  <xacro:arg name='hil_mode' default='false' />
-  <xacro:arg name='hil_state_level' default='false' />
-  <xacro:arg name='vehicle_is_tailsitter' default='false' />
-  <xacro:arg name='visual_material' default='DarkGrey' />
-  <xacro:arg name='enable_mavlink_interface' default='true' />
-  <xacro:arg name='enable_wind' default='false' />
+  <xacro:arg name="name" default="iris" />
+  <xacro:arg name="mavlink_addr" default="INADDR_ANY" />
+  <xacro:arg name="mavlink_udp_port" default="14560" />
+  <xacro:arg name="mavlink_tcp_port" default="4560" />
+  <xacro:arg name="serial_enabled" default="false" />
+  <xacro:arg name="serial_device" default="/dev/ttyACM0" />
+  <xacro:arg name="baudrate" default="921600" />
+  <xacro:arg name="qgc_addr" default="INADDR_ANY" />
+  <xacro:arg name="qgc_udp_port" default="14550" />
+  <xacro:arg name="hil_mode" default="false" />
+  <xacro:arg name="hil_state_level" default="false" />
+  <xacro:arg name="send_vision_estimation" default="false" />
+  <xacro:arg name="send_odometry" default="false" />
+  <xacro:arg name="enable_lockstep" default="true" />
+  <xacro:arg name="use_tcp" default="true" />
+  <xacro:arg name="vehicle_is_tailsitter" default="false" />
+  <xacro:arg name="visual_material" default="DarkGrey" />
+  <xacro:arg name="enable_mavlink_interface" default="true" />
+  <xacro:arg name="enable_wind" default="false" />
   <!-- The following causes segfault with multiple vehicles if defaults to true!!! -->
-  <xacro:arg name='enable_ground_truth' default='false' />
-  <xacro:arg name='enable_logging' default='false' />
-  <xacro:arg name='log_file' default='iris' />
+  <xacro:arg name="enable_ground_truth" default="false" />
+  <xacro:arg name="enable_logging" default="false" />
+  <xacro:arg name="log_file" default="iris" />
   <!-- macros for gazebo plugins, sensors -->
   <xacro:include filename="$(find intel_aero_description)/urdf/component_snippets.xacro" />
   <!-- Instantiate iris "mechanics" -->
   <xacro:include filename="$(find intel_aero_description)/urdf/iris.xacro" />
-  <xacro:if value="$(arg enable_wind)">
-    <xacro:wind_plugin_macro
+  <!-- Only instantiate sensors, Mavlink, etc. if running full SITL simulation -->
+  <xacro:unless value="$(arg spawn_only)">
+    <xacro:if value="$(arg enable_wind)">
+      <xacro:wind_plugin_macro
+          namespace="$(arg namespace)"
+          wind_direction="0 0 1"
+          wind_force_mean="0.7"
+          xyz_offset="1 0 0"
+          wind_gust_direction="0 0 0"
+          wind_gust_duration="0"
+          wind_gust_start="0"
+          wind_gust_force_mean="0"
+          />
+    </xacro:if>
+    <!-- Instantiate gps plugin. -->
+    <xacro:gps_plugin_macro namespace="$(arg namespace)" gps_noise="false" />
+    <xacro:if value="$(arg enable_mavlink_interface)">
+      <!-- Instantiate mavlink telemetry interface. -->
+      <xacro:mavlink_interface_macro
+          namespace="$(arg namespace)"
+          imu_sub_topic="/imu"
+          gps_sub_topic="/gps"
+          mavlink_addr="$(arg mavlink_addr)"
+          mavlink_udp_port="$(arg mavlink_udp_port)"
+          mavlink_tcp_port="$(arg mavlink_tcp_port)"
+          serial_enabled="$(arg serial_enabled)"
+          serial_device="$(arg serial_device)"
+          baudrate="$(arg baudrate)"
+          qgc_addr="$(arg qgc_addr)"
+          qgc_udp_port="$(arg qgc_udp_port)"
+          hil_mode="$(arg hil_mode)"
+          hil_state_level="$(arg hil_state_level)"
+          vehicle_is_tailsitter="$(arg vehicle_is_tailsitter)"
+          send_vision_estimation="$(arg send_vision_estimation)"
+          send_odometry="$(arg send_odometry)"
+          enable_lockstep="$(arg enable_lockstep)"
+          use_tcp="$(arg use_tcp)"
+          >
+      </xacro:mavlink_interface_macro>
+    </xacro:if>
+    <!-- Mount an ADIS16448 IMU. -->
+    <xacro:imu_plugin_macro
         namespace="$(arg namespace)"
-        wind_direction="0 0 1"
-        wind_force_mean="0.7"
-        xyz_offset="1 0 0"
-        wind_gust_direction="0 0 0"
-        wind_gust_duration="0"
-        wind_gust_start="0"
-        wind_gust_force_mean="0"
-        />
-  </xacro:if>
-  <!-- Instantiate gps plugin. -->
-  <xacro:gps_plugin_macro namespace="$(arg namespace)" gps_noise="false" />
-  <!-- Instantiate mavlink telemetry interface. -->
-  <xacro:if value="$(arg enable_mavlink_interface)">
-    <xacro:mavlink_interface_macro
-      namespace="$(arg namespace)"
-      imu_sub_topic="/imu"
-      gps_sub_topic="/gps"
-      mavlink_addr="$(arg mavlink_addr)"
-      mavlink_udp_port="$(arg mavlink_udp_port)"
-      serial_enabled="$(arg serial_enabled)"
-      serial_device="$(arg serial_device)"
-      baudrate="$(arg baudrate)"
-      qgc_addr="$(arg qgc_addr)"
-      qgc_udp_port="$(arg qgc_udp_port)"
-      hil_mode="$(arg hil_mode)"
-      hil_state_level="$(arg hil_state_level)"
-      vehicle_is_tailsitter="$(arg vehicle_is_tailsitter)"
-      >
-    </xacro:mavlink_interface_macro>
-  </xacro:if>
-  <!-- Mount an ADIS16448 IMU. -->
-  <xacro:imu_plugin_macro
-    namespace="$(arg namespace)"
-    imu_suffix=""
-    parent_link="$(arg namespace)/base_link"
-    imu_topic="/imu"
-    mass_imu_sensor="0.015"
-    gyroscope_noise_density="0.0003394"
-    gyroscopoe_random_walk="0.000038785"
-    gyroscope_bias_correlation_time="1000.0"
-    gyroscope_turn_on_bias_sigma="0.0087"
-    accelerometer_noise_density="0.004"
-    accelerometer_random_walk="0.006"
-    accelerometer_bias_correlation_time="300.0"
-    accelerometer_turn_on_bias_sigma="0.1960"
-  >
-    <inertia ixx="0.00001" ixy="0.0" ixz="0.0" iyy="0.00001" iyz="0.0" izz="0.00001" />
-    <origin xyz="0 0 0" rpy="0 0 0" />
-  </xacro:imu_plugin_macro>
-  <xacro:if value="$(arg enable_ground_truth)">
-    <!-- Mount an IMU providing ground truth. -->
-    <xacro:imu_plugin_macro
-      namespace="$(arg namespace)"
-      imu_suffix="gt"
-      parent_link="$(arg namespace)/base_link"
-      imu_topic="ground_truth/imu"
-      mass_imu_sensor="0.00001"
-      gyroscope_noise_density="0.0"
-      gyroscopoe_random_walk="0.0"
-      gyroscope_bias_correlation_time="1000.0"
-      gyroscope_turn_on_bias_sigma="0.0"
-      accelerometer_noise_density="0.0"
-      accelerometer_random_walk="0.0"
-      accelerometer_bias_correlation_time="300.0"
-      accelerometer_turn_on_bias_sigma="0.0"
-    >
+        imu_suffix=""
+        parent_link="$(arg namespace)/base_link"
+        imu_topic="/imu"
+        mass_imu_sensor="0.015"
+        gyroscope_noise_density="0.0003394"
+        gyroscopoe_random_walk="0.000038785"
+        gyroscope_bias_correlation_time="1000.0"
+        gyroscope_turn_on_bias_sigma="0.0087"
+        accelerometer_noise_density="0.004"
+        accelerometer_random_walk="0.006"
+        accelerometer_bias_correlation_time="300.0"
+        accelerometer_turn_on_bias_sigma="0.1960"
+        >
       <inertia ixx="0.00001" ixy="0.0" ixz="0.0" iyy="0.00001" iyz="0.0" izz="0.00001" />
       <origin xyz="0 0 0" rpy="0 0 0" />
     </xacro:imu_plugin_macro>
-    <!-- Mount a generic odometry sensor providing ground truth. -->
-    <xacro:odometry_plugin_macro
-      namespace="$(arg namespace)/ground_truth"
-      odometry_sensor_suffix="gt"
-      parent_link="$(arg namespace)/base_link"
-      pose_topic="pose"
-      pose_with_covariance_topic="pose_with_covariance"
-      position_topic="position"
-      transform_topic="transform"
-      odometry_topic="odometry"
-      parent_frame_id="world"
-      mass_odometry_sensor="0.00001"
-      measurement_divisor="1"
-      measurement_delay="0"
-      unknown_delay="0.0"
-      noise_normal_position="0 0 0"
-      noise_normal_quaternion="0 0 0"
-      noise_normal_linear_velocity="0 0 0"
-      noise_normal_angular_velocity="0 0 0"
-      noise_uniform_position="0 0 0"
-      noise_uniform_quaternion="0 0 0"
-      noise_uniform_linear_velocity="0 0 0"
-      noise_uniform_angular_velocity="0 0 0"
-      enable_odometry_map="false"
-      odometry_map=""
-      image_scale=""
-    >
-      <inertia ixx="0.00001" ixy="0.0" ixz="0.0" iyy="0.00001" iyz="0.0" izz="0.00001" /> <!-- [kg.m^2] [kg.m^2] [kg.m^2] [kg.m^2] [kg.m^2] [kg.m^2] -->
-      <origin xyz="0.0 0.0 0.0" rpy="0.0 0.0 0.0" />
-    </xacro:odometry_plugin_macro>
-  </xacro:if>
-  <xacro:if value="$(arg enable_logging)">
-    <!-- Instantiate a logger -->
-    <xacro:bag_plugin_macro
-      namespace="$(arg namespace)"
-      bag_file="$(arg log_file)"
-      rotor_velocity_slowdown_sim="${rotor_velocity_slowdown_sim}"
-    >
-    </xacro:bag_plugin_macro>
-  </xacro:if>
+    <xacro:if value="$(arg enable_ground_truth)">
+      <!-- Mount an IMU providing ground truth. -->
+      <xacro:imu_plugin_macro
+          namespace="$(arg namespace)"
+          imu_suffix="gt"
+          parent_link="$(arg namespace)/base_link"
+          imu_topic="ground_truth/imu"
+          mass_imu_sensor="0.00001"
+          gyroscope_noise_density="0.0"
+          gyroscopoe_random_walk="0.0"
+          gyroscope_bias_correlation_time="1000.0"
+          gyroscope_turn_on_bias_sigma="0.0"
+          accelerometer_noise_density="0.0"
+          accelerometer_random_walk="0.0"
+          accelerometer_bias_correlation_time="300.0"
+          accelerometer_turn_on_bias_sigma="0.0"
+          >
+        <inertia ixx="0.00001" ixy="0.0" ixz="0.0" iyy="0.00001" iyz="0.0" izz="0.00001" />
+        <origin xyz="0 0 0" rpy="0 0 0" />
+      </xacro:imu_plugin_macro>
+      <!-- Mount a generic odometry sensor providing ground truth. -->
+      <xacro:odometry_plugin_macro
+          namespace="$(arg namespace)/ground_truth"
+          odometry_sensor_suffix="gt"
+          parent_link="$(arg namespace)/base_link"
+          pose_topic="pose"
+          pose_with_covariance_topic="pose_with_covariance"
+          position_topic="position"
+          transform_topic="transform"
+          odometry_topic="odometry"
+          parent_frame_id="world"
+          mass_odometry_sensor="0.00001"
+          measurement_divisor="1"
+          measurement_delay="0"
+          unknown_delay="0.0"
+          noise_normal_position="0 0 0"
+          noise_normal_quaternion="0 0 0"
+          noise_normal_linear_velocity="0 0 0"
+          noise_normal_angular_velocity="0 0 0"
+          noise_uniform_position="0 0 0"
+          noise_uniform_quaternion="0 0 0"
+          noise_uniform_linear_velocity="0 0 0"
+          noise_uniform_angular_velocity="0 0 0"
+          enable_odometry_map="false"
+          odometry_map=""
+          image_scale=""
+          >
+        <inertia ixx="0.00001" ixy="0.0" ixz="0.0" iyy="0.00001" iyz="0.0" izz="0.00001" /> <!-- [kg.m^2] [kg.m^2] [kg.m^2] [kg.m^2] [kg.m^2] [kg.m^2] -->
+        <origin xyz="0.0 0.0 0.0" rpy="0.0 0.0 0.0" />
+      </xacro:odometry_plugin_macro>
+    </xacro:if>
+    <xacro:if value="$(arg enable_logging)">
+      <!-- Instantiate a logger -->
+      <xacro:bag_plugin_macro
+          namespace="$(arg namespace)"
+          bag_file="$(arg log_file)"
+          rotor_velocity_slowdown_sim="${rotor_velocity_slowdown_sim}"
+          >
+      </xacro:bag_plugin_macro>
+    </xacro:if>
+  </xacro:unless>
 </robot>
